File: blackbody_c/hw/blackbody_c.kicad_sch (KiCad schematic)
At the start: 7 parts, among them IC101 TSL25911FN

Commit message: blackbody c revisions based on review
Parts:
- IC101: footprint footprints:TSL25911FN -> footprints:ams_TSL25911FN; symbol TSL25911FN:TSL25911FN -> ams_TSL25911FN:TSL25911FN
Changed lines of the file:
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@@
     )
   )
-  (symbol (lib_id "TSL25911FN:TSL25911FN") (at 113.03 90.17 0) (unit 1)
+  (symbol (lib_id "ams_TSL25911FN:TSL25911FN") (at 113.03 90.17 0) (unit 1)
     (in_bom yes) (on_board yes) (dnp no) (fields_autoplaced)
     (property "Reference" "IC101" (at 125.73 82.55 0)
@@
       (effects (font (size 1.27 1.27)))
     )
-    (property "Footprint" "footprints:TSL25911FN" (at 134.62 185.09 0)
+    (property "Footprint" "footprints:ams_TSL25911FN" (at 134.62 185.09 0)
       (effects (font (size 1.27 1.27)) (justify left top) hide)
     )

Commit message: fixes for blackbody b before prod
Parts:
- C101: Cost 0.0037 -> 0.10; Distributor JLCPCB -> Mouser; LCSC Part # C52923 -> (none); Manufacturer Samsung Electro-Mechanics -> Murata Electronics; P/N CL05A105KA5NQNC -> GRM155R70J105KA2D
- R101: Cost 0.0005 -> 0.57; Distributor JLCPCB -> Mouser; LCSC Part # C11702 -> (none); Manufacturer UNI-ROYAL(Uniroyal Elec) -> Panasonic; P/N 0402WGF1001TCE -> ERA-2ARC102X
Changed lines of the file:
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@@
       (effects (font (size 1.27 1.27)) hide)
     )
-    (property "Datasheet" "https://datasheet.lcsc.com/lcsc/2206010216_UNI-ROYAL-Uniroyal-Elec-0402WGF1001TCE_C11702.pdf" (at 101.6 87.63 0)
+    (property "Datasheet" "https://www.mouser.com/datasheet/2/315/AOA0000C307-1149632.pdf" (at 101.6 87.63 0)
       (effects (font (size 1.27 1.27)) hide)
     )
-    (property "Distributor" "JLCPCB" (at 101.6 87.63 0)
+    (property "Distributor" "Mouser" (at 101.6 87.63 0)
       (effects (font (size 1.27 1.27)) hide)
     )
-    (property "Manufacturer" "UNI-ROYAL(Uniroyal Elec)" (at 101.6 87.63 0)
+    (property "Manufacturer" "Panasonic" (at 101.6 87.63 0)
       (effects (font (size 1.27 1.27)) hide)
     )
-    (property "P/N" "0402WGF1001TCE" (at 101.6 87.63 0)
+    (property "P/N" "ERA-2ARC102X" (at 101.6 87.63 0)
       (effects (font (size 1.27 1.27)) hide)
     )
-    (property "LCSC Part #" "C11702" (at 101.6 87.63 0)
+    (property "LCSC Part #" "" (at 101.6 87.63 0)
       (effects (font (size 1.27 1.27)) hide)
     )
-    (property "Cost" "0.0005" (at 101.6 87.63 0)
+    (property "Cost" "0.57" (at 101.6 87.63 0)
       (effects (font (size 1.27 1.27)) hide)
     )
@@
       (effects (font (size 1.27 1.27)) hide)
     )
-    (property "Datasheet" "https://datasheet.lcsc.com/lcsc/2304140030_Samsung-Electro-Mechanics-CL05A105KA5NQNC_C52923.pdf" (at 161.29 91.44 0)
+    (property "Datasheet" "https://www.mouser.com/datasheet/2/281/1/GRM155R70J105KA12_01A-1984187.pdf" (at 161.29 91.44 0)
       (effects (font (size 1.27 1.27)) hide)
     )
-    (property "Distributor" "JLCPCB" (at 161.29 91.44 0)
+    (property "Distributor" "Mouser" (at 161.29 91.44 0)
       (effects (font (size 1.27 1.27)) hide)
     )
-    (property "Manufacturer" "Samsung Electro-Mechanics" (at 161.29 91.44 0)
+    (property "Manufacturer" "Murata Electronics" (at 161.29 91.44 0)
       (effects (font (size 1.27 1.27)) hide)
     )
-    (property "P/N" "CL05A105KA5NQNC" (at 161.29 91.44 0)
+    (property "P/N" "GRM155R70J105KA2D" (at 161.29 91.44 0)
       (effects (font (size 1.27 1.27)) hide)
     )
-    (property "LCSC Part #" "C52923" (at 161.29 91.44 0)
+    (property "LCSC Part #" "" (at 161.29 91.44 0)
       (effects (font (size 1.27 1.27)) hide)
     )
-    (property "Cost" "0.0037" (at 161.29 91.44 0)
+    (property "Cost" "0.10" (at 161.29 91.44 0)
       (effects (font (size 1.27 1.27)) hide)
     )
