File: blackbody_a/hw/comm_can.kicad_sch (KiCad schematic)
At the start: 22 parts, among them IC401 ADM3055EBRIZ, J401 43650-0427, J402 43650-0427

Commit message: fixes for blackbody b before prod
Parts:
- D401: Cost 0.1982 -> 0.37; Distributor JLCPCB -> Mouser; LCSC Part # C350941 -> (none)
- L2, L3: footprint Inductor_SMD:L_0402_1005Metric -> Resistor_SMD:R_0402_1005Metric; Cost 0.0155 -> 0.10; Distributor JLCPCB -> Mouser; LCSC Part # C2683172 -> (none)
- R10: Cost 0.0005 -> 0.10; Distributor JLCPCB -> Mouser; LCSC Part # C60310 -> (none); Manufacturer UNI-ROYAL(Uniroyal Elec) -> Bourns; P/N 0402WGF604JTCE -> CR0402-FX-60R4GLF
Changed lines of the file:
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@@
       (effects (font (size 1 1)) hide)
     )
-    (property "Distributor" "JLCPCB" (at 194.31 104.14 90)
-      (effects (font (size 1 1)) hide)
-    )
-    (property "Manufacturer" "UNI-ROYAL(Uniroyal Elec)" (at 194.31 104.14 90)
-      (effects (font (size 1 1)) hide)
-    )
-    (property "P/N" "0402WGF604JTCE" (at 194.31 104.14 90)
-      (effects (font (size 1 1)) hide)
-    )
-    (property "LCSC Part #" "C60310" (at 194.31 104.14 90)
-      (effects (font (size 1 1)) hide)
-    )
-    (property "Cost" "0.0005" (at 194.31 104.14 90)
+    (property "Distributor" "Mouser" (at 194.31 104.14 90)
+      (effects (font (size 1 1)) hide)
+    )
+    (property "Manufacturer" "Bourns" (at 194.31 104.14 90)
+      (effects (font (size 1 1)) hide)
+    )
+    (property "P/N" "CR0402-FX-60R4GLF" (at 194.31 104.14 90)
+      (effects (font (size 1 1)) hide)
+    )
+    (property "LCSC Part #" "" (at 194.31 104.14 90)
+      (effects (font (size 1 1)) hide)
+    )
+    (property "Cost" "0.10" (at 194.31 104.14 90)
       (effects (font (size 1 1)) hide)
     )
@@
       (effects (font (size 1 1)) (justify left top) hide)
     )
-    (property "Distributor" "JLCPCB" (at 187.96 121.92 0)
+    (property "Distributor" "Mouser" (at 187.96 121.92 0)
       (effects (font (size 1 1)) hide)
     )
@@
       (effects (font (size 1 1)) hide)
     )
-    (property "LCSC Part #" "C350941" (at 187.96 121.92 0)
-      (effects (font (size 1 1)) hide)
-    )
-    (property "Cost" "0.1982" (at 187.96 121.92 0)
+    (property "LCSC Part #" "" (at 187.96 121.92 0)
+      (effects (font (size 1 1)) hide)
+    )
+    (property "Cost" "0.37" (at 187.96 121.92 0)
       (effects (font (size 1 1)) hide)
     )
@@
       (effects (font (size 1 1)) hide)
     )
-    (property "Distributor" "JLCPCB" (at 184.15 104.14 90)
-      (effects (font (size 1 1)) hide)
-    )
-    (property "Manufacturer" "UNI-ROYAL(Uniroyal Elec)" (at 184.15 104.14 90)
-      (effects (font (size 1 1)) hide)
-    )
-    (property "P/N" "0402WGF604JTCE" (at 184.15 104.14 90)
-      (effects (font (size 1 1)) hide)
-    )
-    (property "LCSC Part #" "C60310" (at 184.15 104.14 90)
-      (effects (font (size 1 1)) hide)
-    )
-    (property "Cost" "0.0005" (at 184.15 104.14 90)
+    (property "Distributor" "Mouser" (at 184.15 104.14 90)
+      (effects (font (size 1 1)) hide)
+    )
+    (property "Manufacturer" "Bourns" (at 184.15 104.14 90)
+      (effects (font (size 1 1)) hide)
+    )
+    (property "P/N" "CR0402-FX-60R4GLF" (at 184.15 104.14 90)
+      (effects (font (size 1 1)) hide)
+    )
+    (property "LCSC Part #" "" (at 184.15 104.14 90)
+      (effects (font (size 1 1)) hide)
+    )
+    (property "Cost" "0.10" (at 184.15 104.14 90)
       (effects (font (size 1 1)) hide)
     )
@@
       (effects (font (size 1 1)) (justify right))
     )
-    (property "Footprint" "Inductor_SMD:L_0402_1005Metric" (at 146.05 92.202 90)
+    (property "Footprint" "Resistor_SMD:R_0402_1005Metric" (at 146.05 92.202 90)
       (effects (font (size 1 1)) hide)
     )
@@
       (effects (font (size 1 1)) hide)
     )
-    (property "Distributor" "JLCPCB" (at 146.05 93.98 90)
+    (property "Distributor" "Mouser" (at 146.05 93.98 90)
       (effects (font (size 1.016 1.016)) hide)
     )
@@
       (effects (font (size 1.016 1.016)) hide)
     )
-    (property "LCSC Part #" "C2683172" (at 146.05 93.98 90)
-      (effects (font (size 1.016 1.016)) hide)
-    )
-    (property "Cost" "0.0155" (at 146.05 93.98 90)
+    (property "LCSC Part #" "" (at 146.05 93.98 90)
+      (effects (font (size 1.016 1.016)) hide)
+    )
+    (property "Cost" "0.10" (at 146.05 93.98 90)
       (effects (font (size 1.016 1.016)) hide)
     )
@@
       (effects (font (size 1 1)) (justify right))
     )
-    (property "Footprint" "Inductor_SMD:L_0402_1005Metric" (at 146.05 97.282 90)
+    (property "Footprint" "Resistor_SMD:R_0402_1005Metric" (at 146.05 97.282 90)
       (effects (font (size 1 1)) hide)
     )
@@
       (effects (font (size 1 1)) hide)
     )
-    (property "Distributor" "JLCPCB" (at 146.05 99.06 90)
+    (property "Distributor" "Mouser" (at 146.05 99.06 90)
       (effects (font (size 1.016 1.016)) hide)
     )
@@
       (effects (font (size 1.016 1.016)) hide)
     )
-    (property "LCSC Part #" "C2683172" (at 146.05 99.06 90)
-      (effects (font (size 1.016 1.016)) hide)
-    )
-    (property "Cost" "0.0155" (at 146.05 99.06 90)
-      (effects (font (size 1.016 1.016)) hide)
-    )
+    (property "LCSC Part #" "" (at 146.05 99.06 90)
+      (effects (font (size 1.016 1.016)) hide)
+    )
+    (property "Cost" "0.10" (at 146.05 99.06 90)
+      (effects (font (size 1.016 1.016)) hide)
+    )
