File: blackbody_a/hw/power_reg.kicad_sch (KiCad schematic)
At the start: 8 parts, among them J301 43650-0227

Commit message: fixes for blackbody b before prod
Parts:
- L301: Cost 0.0781 -> 0.42; Distributor JLCPCB -> Mouser; LCSC Part # C307864 -> (none); Notes Footprint compatible with equivalent VLS252010CX-2R2M-1 on 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 -> (none); P/N VLS252010MNT-2R2M -> VLS252010CX-2R2M-1
- PS301: Cost 1.086 -> 1.63; Distributor TI -> Mouser; Notes Alt distributor: Mouser -> Alt distributor: TI
Changed lines of the file:
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@@
       (effects (font (size 1 1)) hide)
     )
-    (property "Distributor" "TI" (at 139.7 95.25 0)
+    (property "Distributor" "Mouser" (at 139.7 95.25 0)
       (effects (font (size 1 1)) hide)
     )
@@
       (effects (font (size 1 1)) hide)
     )
-    (property "Cost" "1.086" (at 139.7 95.25 0)
+    (property "Cost" "1.63" (at 139.7 95.25 0)
       (effects (font (size 1 1)) hide)
     )
-    (property "Notes" "Alt distributor: Mouser" (at 139.7 95.25 0)
+    (property "Notes" "Alt distributor: TI" (at 139.7 95.25 0)
       (effects (font (size 1 1)) hide)
     )
@@
       (effects (font (size 1 1)) hide)
     )
-    (property "Datasheet" "https://datasheet.lcsc.com/lcsc/2005181102_TDK-VLS252010MNT-2R2M_C307864.pdf" (at 165.1 85.09 0)
+    (property "Datasheet" "https://product.tdk.com/system/files/dam/doc/product/inductor/inductor/smd/catalog/inductor_commercial_power_vls252010cx-1_en.pdf?ref_disty=mouser" (at 165.1 85.09 0)
       (effects (font (size 1 1)) hide)
     )
-    (property "Distributor" "JLCPCB" (at 165.1 85.09 90)
+    (property "Distributor" "Mouser" (at 165.1 85.09 90)
       (effects (font (size 1 1)) hide)
     )
@@
       (effects (font (size 1 1)) hide)
     )
-    (property "P/N" "VLS252010MNT-2R2M" (at 165.1 85.09 90)
+    (property "P/N" "VLS252010CX-2R2M-1" (at 165.1 85.09 90)
       (effects (font (size 1 1)) hide)
     )
-    (property "LCSC Part #" "C307864" (at 165.1 85.09 90)
+    (property "LCSC Part #" "" (at 165.1 85.09 90)
       (effects (font (size 1 1)) hide)
     )
-    (property "Cost" "0.0781" (at 165.1 85.09 90)
+    (property "Cost" "0.42" (at 165.1 85.09 90)
       (effects (font (size 1 1)) hide)
     )
-    (property "Notes" "Footprint compatible with equivalent VLS252010CX-2R2M-1 on Mouser." (at 165.1 85.09 90)
+    (property "Notes" "" (at 165.1 85.09 90)
       (effects (font (size 1 1)) hide)
     )
